File: PDPowerSupply.kicad_sch (KiCad schematic)
At the start: 29 parts, among them J1 USB_C_Receptacle_USB2.0_16P, J2 Barrel_Jack_Switch, J3 Barrel_Jack_Switch, J4 Barrel_Jack_Switch, J5 Barrel_Jack_Switch, J6 Barrel_Jack_Switch, J7 Barrel_Jack_Switch, J8 Barrel_Jack_Switch, Q2 Q_PMOS_GDS, U1 CH224K

Commit message: v2.0発注
Parts:
- removed TP1, TP2, TP4: TestPoint, TestPoint:TestPoint_THTPad_D1.5mm_Drill0.7mm, symbol Connector:TestPoint
- added D3: VDD_LED, LED_SMD:LED_0603_1608Metric_Pad1.05x0.95mm_HandSolder, symbol Device:LED_Small
- added R6: 470R, Capacitor_SMD:C_0603_1608Metric_Pad1.08x0.95mm_HandSolder, symbol Device:R_Small
- added SW1: SW_SPDT, Ishihalib:ROCKERSW_3MS1J102M2QES, symbol Switch:SW_SPDT
Connections:
- net +9V: now also C3.1, SW1.1 (A); no longer Q2.2 (D)
- net GND: now also R6.2
- net JACK_B: now reaches J8.3
- net JACK_B: now also Q2.2 (D)
- net at F1.2, Q2.3 (S), R1.1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: no longer C3.1
- net VBUS: no longer names the net of F1.1, J1.A4 (VBUS), J1.A9 (VBUS), J1.B4 (VBUS), J1.B9 (VBUS)
- net VBUS: no longer J8.2
- new net: D3.1 (K), R6.1
- new net VDD: D3.2 (A), J8.2, SW1.2 (B)
Other:
- moved on the sheet: C3, D1
